File: Untitled.sch (KiCad schematic (older format))
At the start: 17 parts

Commit message: Add resistor
Parts:
- added R?: R, symbol Device:R
Connections:
- wire segments 62 -> 63
Changed lines of the file:
@@
 	1750 2250 2100 2250
 Wire Wire Line
-	2100 2250 2100 3000
+	2100 2250 2100 2450
 Wire Wire Line
 	2100 3300 2100 3850
+$Comp
+L Device:R R?
+U 1 1 5E63D44D
+P 2100 2600
+F 0 "R?" V 1893 2600 50  0000 C CNN
+F 1 "R" V 1984 2600 50  0000 C CNN
+F 2 "" V 2030 2600 50  0001 C CNN
+F 3 "~" H 2100 2600 50  0001 C CNN
+	1    2100 2600
+	-1   0    0    1
+$EndComp
+Wire Wire Line
+	2100 2750 2100 3000
 $EndSCHEMATC
